Commit message: Changes orientation to face positive x with boxer.

File: forwardkinematics/urdfFks/urdf/boxer.urdf (robot description, URDF)
Before this commit: robot albert, 6 links, 5 joints
Links:
- added link base_link_ori
Joints:
- added joint base_add_orientation: type fixed, parent base_link_ori, child base_link, origin xyz=0.0 0 0 rpy=0 0 1.57079
- joint ee_joint: origin xyz=0.4 0 0 rpy=0 0 0 -> xyz=0 -0.4 0 rpy=0 0 0; parent chassis_link -> base_link
- joint world_base_theta: child base_link -> base_link_ori
