Commit message: Adds tiago fk.

File: forwardkinematics/urdfFks/urdf/tiago.urdf (robot description, URDF)
Before this commit: robot tiago_dual, 49 links, 48 joints
Links:
- added link base_link_ori
- added link world
- added link world_base_link_x
- added link world_base_link_y
- link arm_left_1_link: geometry 
- link arm_left_2_link: geometry 
- link arm_left_3_link: geometry 
- link arm_left_4_link: geometry 
- link arm_left_5_link: geometry 
- link arm_left_6_link: geometry 
- link arm_left_tool_link: geometry 
- link arm_right_1_link: geometry 
- link arm_right_2_link: geometry 
- link arm_right_3_link: geometry 
- link arm_right_4_link: geometry 
- link arm_right_5_link: geometry 
- link arm_right_6_link: geometry 
- link arm_right_tool_link: geometry 
- link base_link: geometry 
- link caster_back_left_1_link: geometry 
- link caster_back_left_2_link: geometry 
- link caster_back_right_1_link: geometry 
- link caster_back_right_2_link: geometry 
- link caster_front_left_1_link: geometry 
- link caster_front_left_2_link: geometry 
- link caster_front_right_1_link: geometry 
- link caster_front_right_2_link: geometry 
- link gripper_left_left_finger_link: geometry 
- link gripper_left_link: geometry 
- link gripper_left_right_finger_link: geometry 
- link gripper_right_left_finger_link: geometry 
- link gripper_right_link: geometry 
- link gripper_right_right_finger_link: geometry 
- link head_1_link: geometry 
- link head_2_link: geometry 
- link torso_fixed_column_link: geometry 
- link torso_fixed_link: geometry 
- link torso_lift_link: geometry 
- link wheel_left_link: geometry 
- link wheel_right_link: geometry 
- link wrist_left_ft_link: geometry 
- link wrist_left_ft_tool_link: geometry 
- link wrist_right_ft_link: geometry 
- link wrist_right_ft_tool_link: geometry 
- link xtion_link: geometry 
Joints:
- added joint base_add_orientation: type fixed, parent base_link_ori, child base_link, origin xyz=0.0 0 0 rpy=0 0 0
- added joint world_base_theta: type revolute, parent world_base_link_y, child base_link_ori, origin xyz=0 0 0 rpy=0 0 0, axis 0 0 1, limit lower=-15 upper=15 effort=100 velocity=5
- added joint world_base_x: type prismatic, parent world, child world_base_link_x, origin xyz=0 0 0 rpy=0 0 0, axis 1 0 0, limit lower=-15 upper=15 effort=100 velocity=5
- added joint world_base_y: type prismatic, parent world_base_link_x, child world_base_link_y, origin xyz=0 0 0 rpy=0 0 0, axis 0 1 0, limit lower=-15 upper=15 effort=100 velocity=5

Commit message: Correct tiago fk using the gym environment.

File: forwardkinematics/urdfFks/urdf/tiago.urdf (robot description, URDF)
Before this commit: robot tiago_dual, 53 links, 52 joints
Joints:
- joint base_add_orientation: origin xyz=0.0 0 0 rpy=0 0 0 -> xyz=-0.18 0 0.10 rpy=0 0 0
- joint gripper_left_grasping_frame_joint: origin xyz=0 0 -0.12 rpy=-1.5708 1.5708 0 -> xyz=0 0 -0.20 rpy=-1.5708 1.5708 0
- joint gripper_right_grasping_frame_joint: origin xyz=0 0 -0.12 rpy=-1.5708 1.5708 0 -> xyz=0 0 -0.20 rpy=-1.5708 1.5708 0
