Commit message: Adds origin for non-holonomic fks.

File: forwardkinematics/urdfFks/urdf/pointRobot.urdf (robot description, URDF)
Before this commit: robot pointRobot, 4 links, 3 joints
Links:
- added link origin
Joints:
- added joint boxer_joint_world: type fixed, parent world, child origin, origin xyz=0 0 0 rpy=0 0 0
- joint mobile_joint_x: parent world -> origin
