Commit message: Simplifies albertFk by removing meshes. Adds link9 for end-effector.

File: forwardkinematics/urdfFks/urdf/albert.urdf (robot description, URDF)
Before this commit: robot albert, 34 links, 33 joints
Links:
- removed link base_footprint
- removed link chassis_link
- removed link extrusion2
- removed link extrusion3
- removed link extrusion4
- removed link front_laser
- removed link imu_link
- removed link rear_left_sonar_link
- removed link rear_right_sonar_link
- removed link rotacastor_left_link
- removed link rotacastor_right_link
- removed link stereo
- removed link stereo_left
- removed link stereo_right
- removed link wheel_left_link
- removed link wheel_right_link
- added link mmrobot_link9
- added link world
- added link world_baske_link_x
- added link world_baske_link_y
- link extrusion1: geometry 
- link internal_link: geometry 
- link lift_link: geometry 
- link mmrobot_hand: geometry 
- link mmrobot_leftfinger: geometry 
- link mmrobot_link0: geometry 
- link mmrobot_link1: geometry 
- link mmrobot_link2: geometry 
- link mmrobot_link3: geometry 
- link mmrobot_link4: geometry 
- link mmrobot_link5: geometry 
- link mmrobot_link6: geometry 
- link mmrobot_link7: geometry 
- link mmrobot_rightfinger: geometry 
- link top_mount: geometry 
- link top_mount_bottom: geometry 
Joints:
- removed joint base_footprint_joint
- removed joint base_laser_joint
- removed joint extrusion2_joint
- removed joint extrusion3_joint
- removed joint extrusion4_joint
- removed joint imu_joint
- removed joint rear_left_sonar_joint
- removed joint rear_right_sonar_joint
- removed joint rotacastor_left_joint
- removed joint rotacastor_right_joint
- removed joint stereo_camera_joint
- removed joint stereo_left_joint
- removed joint stereo_right_joint
- removed joint wheel_left_joint
- removed joint wheel_right_joint
- added joint mmrobot_joint9: type fixed, parent mmrobot_link8, child mmrobot_link9, origin xyz=0 0 0.020 rpy=0 0 0, axis 0 0 0
- added joint world_base_theta: type revolute, parent world_base_link_y, child base_link, origin xyz=0 0 0 rpy=0 0 0, axis 0 0 1, limit lower=-15 upper=15 effort=100 velocity=5
- added joint world_base_x: type prismatic, parent world, child world_base_link_x, origin xyz=0 0 0 rpy=0 0 0, axis 1 0 0, limit lower=-15 upper=15 effort=100 velocity=5
- added joint world_base_y: type prismatic, parent world_base_link_x, child world_base_link_y, origin xyz=0 0 0 rpy=0 0 0, axis 0 1 0, limit lower=-15 upper=15 effort=100 velocity=5
- joint lift_joint: type prismatic -> fixed

Commit message: Adds base end-effector for albert. Alligning with boxer.

File: forwardkinematics/urdfFks/urdf/albert.urdf (robot description, URDF)
Before this commit: robot albert, 22 links, 22 joints
Links:
- added link base_tip_link; visual sphere radius=0.0625
Joints:
- added joint base_tip_joint: type fixed, parent base_link, child base_tip_link, origin xyz=0 -0.4 0 rpy=0 0 0

Commit message: Copies panda part to albert urdf and changes AlbertFk accordingly.

File: forwardkinematics/urdfFks/urdf/albert.urdf (robot description, URDF)
Before this commit: robot albert, 23 links, 23 joints
Links:
- removed link mmrobot_hand
- removed link mmrobot_leftfinger
- removed link mmrobot_link0
- removed link mmrobot_link1
- removed link mmrobot_link2
- removed link mmrobot_link3
- removed link mmrobot_link4
- removed link mmrobot_link5
- removed link mmrobot_link6
- removed link mmrobot_link7
- removed link mmrobot_link8
- removed link mmrobot_link9
- removed link mmrobot_rightfinger
- added link panda_hand, mass 0.68; collision mesh filename=meshes/collision/hand.stl; visual mesh filename=meshes/visual/hand.dae
- added link panda_leftfinger, mass 0.01; collision mesh filename=meshes/collision/finger.stl; visual mesh filename=meshes/visual/finger.dae
- added link panda_link0, mass 2.92; collision mesh filename=meshes/collision/link0.stl; visual mesh filename=meshes/visual/link0.dae
- added link panda_link1, mass 2.74; collision mesh filename=meshes/collision/link1.stl; visual mesh filename=meshes/visual/link1.dae
- added link panda_link2, mass 2.74; collision mesh filename=meshes/collision/link2.stl; visual mesh filename=meshes/visual/link2.dae
- added link panda_link3, mass 2.38; collision mesh filename=meshes/collision/link3.stl; visual mesh filename=meshes/visual/link3.dae
- added link panda_link4, mass 2.38; collision mesh filename=meshes/collision/link4.stl; visual mesh filename=meshes/visual/link4.dae
- added link panda_link5, mass 2.74; collision mesh filename=meshes/collision/link5.stl; visual mesh filename=meshes/visual/link5.dae
- added link panda_link6, mass 1.55; collision mesh filename=meshes/collision/link6.stl; visual mesh filename=meshes/visual/link6.dae
- added link panda_link7, mass 0.54; collision mesh filename=meshes/collision/link7.stl; visual mesh filename=meshes/visual/link7.dae
- added link panda_link8
- added link panda_link9
- added link panda_rightfinger, mass 0.01; collision mesh filename=meshes/collision/finger.stl; visual mesh filename=meshes/visual/finger.dae
Joints:
- removed joint mmrobot_finger_joint1
- removed joint mmrobot_finger_joint2
- removed joint mmrobot_hand_joint
- removed joint mmrobot_joint1
- removed joint mmrobot_joint2
- removed joint mmrobot_joint3
- removed joint mmrobot_joint4
- removed joint mmrobot_joint5
- removed joint mmrobot_joint6
- removed joint mmrobot_joint7
- removed joint mmrobot_joint8
- removed joint mmrobot_joint9
- removed joint mmrobot_joint_top_mount
- added joint panda_finger_joint1: type prismatic, parent panda_hand, child panda_leftfinger, origin xyz=0 0 0.0584 rpy=0 0 0, axis 0 1 0, limit lower=0.0 upper=0.04 effort=20 velocity=0.2
- added joint panda_finger_joint2: type prismatic, parent panda_hand, child panda_rightfinger, origin xyz=0 0 0.0584 rpy=0 0 0, axis 0 -1 0, limit lower=0.0 upper=0.04 effort=20 velocity=0.2
- added joint panda_hand_joint: type fixed, parent panda_link8, child panda_hand, origin xyz=0 0 0 rpy=0 0 -0.785398163397
- added joint panda_joint1: type revolute, parent panda_link0, child panda_link1, origin xyz=0 0 0.333 rpy=0 0 0, axis 0 0 1, limit lower=-2.8973 upper=2.8973 effort=87 velocity=2.1750
- added joint panda_joint2: type revolute, parent panda_link1, child panda_link2, origin xyz=0 0 0 rpy=-1.57079632679 0 0, axis 0 0 1, limit lower=-1.7628 upper=1.7628 effort=87 velocity=2.1750
- added joint panda_joint3: type revolute, parent panda_link2, child panda_link3, origin xyz=0 -0.316 0 rpy=1.57079632679 0 0, axis 0 0 1, limit lower=-2.8973 upper=2.8973 effort=87 velocity=2.1750
- added joint panda_joint4: type revolute, parent panda_link3, child panda_link4, origin xyz=0.0825 0 0 rpy=1.57079632679 0 0, axis 0 0 1, limit lower=-3.0718 upper=0.0698 effort=87 velocity=2.1750
- added joint panda_joint5: type revolute, parent panda_link4, child panda_link5, origin xyz=-0.0825 0.384 0 rpy=-1.57079632679 0 0, axis 0 0 1, limit lower=-2.8973 upper=2.8973 effort=12 velocity=2.6100
- added joint panda_joint6: type revolute, parent panda_link5, child panda_link6, origin xyz=0 0 0 rpy=1.57079632679 0 0, axis 0 0 1, limit lower=-0.0175 upper=3.7525 effort=12 velocity=2.6100
- added joint panda_joint7: type revolute, parent panda_link6, child panda_link7, origin xyz=0.088 0 0 rpy=1.57079632679 0 0, axis 0 0 1, limit lower=-2.8973 upper=2.8973 effort=12 velocity=2.6100
- added joint panda_joint8: type fixed, parent panda_link7, child panda_link8, origin xyz=0 0 0.107 rpy=0 0 0, axis 0 0 0
- added joint panda_joint9: type fixed, parent panda_link8, child panda_link9, origin xyz=0 0 0.020 rpy=0 0 0, axis 0 0 0
- added joint panda_joint_top_mount: type fixed, parent top_mount, child panda_link0, origin xyz=-0.15 0 0 rpy=0 0 0

Commit message: Removes meshes from boxer and albert and corrects error in forward kinematics albert due to urdf error.

File: forwardkinematics/urdfFks/urdf/albert.urdf (robot description, URDF)
Before this commit: robot albert, 23 links, 23 joints
Links:
- removed link world_baske_link_x
- removed link world_baske_link_y
- added link chassis_link
- added link world_base_link_x
- added link world_base_link_y
- link base_link: mass 1 -> None
- link base_tip_link: geometry 
- link extrusion1: mass 1 -> None
- link internal_link: mass 31 -> None
- link lift_link: mass 10 -> None
- link panda_hand: mass 0.68 -> None; geometry 
- link panda_leftfinger: mass 0.01 -> None; geometry 
- link panda_link0: mass 2.92 -> None; geometry 
- link panda_link1: mass 2.74 -> None; geometry 
- link panda_link2: mass 2.74 -> None; geometry 
- link panda_link3: mass 2.38 -> None; geometry 
- link panda_link4: mass 2.38 -> None; geometry 
- link panda_link5: mass 2.74 -> None; geometry 
- link panda_link6: mass 1.55 -> None; geometry 
- link panda_link7: mass 0.54 -> None; geometry 
- link panda_rightfinger: mass 0.01 -> None; geometry 
- link top_mount: mass 10 -> None
Joints:
- joint base_chassis_joint: origin xyz=0.15 0 0 rpy=0 0 1.5708 -> xyz=0.0 0 0 rpy=0 0 -1.5708
- joint base_tip_joint: origin xyz=0 -0.4 0 rpy=0 0 0 -> xyz=0.4 0 0 rpy=0 0 0; parent base_link -> chassis_link
- joint internal_joint: origin xyz=0 0 0 rpy=1.5708 0 0 -> xyz=0 0 0 rpy=1.5708 0 1.5708
- joint lift_joint: origin xyz=0 0 0.177 rpy=1.5708 0 0 -> xyz=0 0 0.177 rpy=1.5708 0 1.5708

File: forwardkinematics/urdfFks/urdf/boxer.urdf (robot description, URDF)
Before this commit: robot albert, 5 links, 4 joints
Links:
- removed link world_baske_link_x
- removed link world_baske_link_y
- added link chassis_link
- added link world_base_link_x
- added link world_base_link_y
- link ee_link: geometry 
Joints:
- added joint base_chassis_joint: type fixed, parent base_link, child chassis_link, origin xyz=0.0 0 0 rpy=0 0 -1.5708
- joint ee_joint: origin xyz=0 -0.4 0 rpy=0 0 0 -> xyz=0.4 0 0 rpy=0 0 0; parent base_link -> chassis_link

Commit message: Rotates forward kinematics albert.

File: forwardkinematics/urdfFks/urdf/albert.urdf (robot description, URDF)
Before this commit: robot albert, 24 links, 23 joints
Links:
- added link base_link_ori
Joints:
- added joint base_add_orientation: type fixed, parent base_link_ori, child base_link, origin xyz=0.0 0 0 rpy=0 0 1.57079
- joint world_base_theta: child base_link -> base_link_ori

Commit message: Finishes dual arm and changes tests.

File: forwardkinematics/urdfFks/urdf/albert.urdf (robot description, URDF)
Before this commit: robot albert, 25 links, 24 joints
Joints:
- joint panda_finger_joint1: type prismatic -> fixed
- joint panda_finger_joint2: type prismatic -> fixed

File: forwardkinematics/urdfFks/urdf/panda.urdf (robot description, URDF)
Before this commit: robot panda, 14 links, 13 joints
Joints:
- joint panda_finger_joint1: type prismatic -> fixed
- joint panda_finger_joint2: type prismatic -> fixed

File: forwardkinematics/urdfFks/urdf/tiago.urdf (robot description, URDF)
Before this commit: robot tiago_dual, 53 links, 52 joints
Joints:
- joint gripper_left_left_finger_joint: type prismatic -> fixed
- joint gripper_left_right_finger_joint: type prismatic -> fixed
- joint gripper_right_left_finger_joint: type prismatic -> fixed
- joint gripper_right_right_finger_joint: type prismatic -> fixed

Commit message: Adds origin link in non-holonomic urdfs.

File: forwardkinematics/urdfFks/urdf/albert.urdf (robot description, URDF)
Before this commit: robot albert, 25 links, 24 joints
Links:
- added link origin
Joints:
- added joint boxer_joint_world: type fixed, parent world, child origin, origin xyz=0 0 0 rpy=0 0 0
- joint world_base_x: parent world -> origin

File: forwardkinematics/urdfFks/urdf/boxer.urdf (robot description, URDF)
Before this commit: robot albert, 7 links, 6 joints
Links:
- added link origin
Joints:
- added joint boxer_joint_world: type fixed, parent world, child origin, origin xyz=0 0 0 rpy=0 0 0
- joint world_base_x: parent world -> origin

File: forwardkinematics/urdfFks/urdf/tiago.urdf (robot description, URDF)
Before this commit: robot tiago_dual, 53 links, 52 joints
Links:
- added link origin
Joints:
- added joint boxer_joint_world: type fixed, parent world, child origin, origin xyz=0 0 0 rpy=0 0 0
- joint world_base_x: parent world -> origin

Commit message: ft[generic]: Adds generic fk for diffdrive.
Adding generic fk for diff drive robots. If the base_type is specified
to be `diffdrive`, three additional degrees of freedom are addedd.
Removes orientation correction joint for boxer and albert.

File: forwardkinematics/urdfFks/urdf/albert.urdf (robot description, URDF)
Before this commit: robot albert, 26 links, 25 joints
Links:
- removed link base_link_ori
Joints:
- removed joint base_add_orientation
- joint world_base_theta: child base_link_ori -> base_link

File: forwardkinematics/urdfFks/urdf/boxer.urdf (robot description, URDF)
Before this commit: robot boxer, 8 links, 7 joints
Links:
- removed link base_link_ori
Joints:
- removed joint base_add_orientation
- joint world_base_theta: child base_link_ori -> base_link
